File: bppy/BPN/BPN.kicad_sch (KiCad schematic)
At the start: 33 parts, among them J1 USB_C_Receptacle_PowerOnly_6P, J2 Valve, J3 Pumpe, Q1 2N2219, Q2 IRLIZ44N, U1 LM317_TO-220, U2 NCP1117-3.3_SOT223, U3 Pico, U4 NJM4560, U5 AMS6915

Commit message: with simulator
Parts:
- removed C1: C_Polarized, Capacitor_SMD:CP_Elec_3x5.3, symbol Device:C_Polarized
- removed C3: 10u, Capacitor_SMD:CP_Elec_3x5.3, symbol Device:C_Small
- removed U2: NCP1117-3.3_SOT223, Package_TO_SOT_SMD:SOT-223, symbol Regulator_Linear:NCP1117-3.3_SOT223
- added C1: 0.1u, Capacitor_SMD:C_0805_2012Metric_Pad1.18x1.45mm_HandSolder, symbol Device:C_Small
- added D2: 1N4002, Diode_THT:D_DO-41_SOD81_P3.81mm_Vertical_AnodeUp, symbol Diode:1N4002
- added J4: Sensor_2, Connector_PinSocket_2.54mm:PinSocket_1x06_P2.54mm_Vertical, symbol Connector:Conn_01x06_Socket
- C2: value 10u -> 1u; footprint Capacitor_SMD:CP_Elec_3x5.3 -> Capacitor_SMD:C_0805_2012Metric_Pad1.18x1.45mm_HandSolder
- C3: renamed from C4; footprint Capacitor_SMD:CP_Elec_3x5.3 -> Capacitor_SMD:C_0805_2012Metric_Pad1.18x1.45mm_HandSolder
- C4: renamed from C5; footprint Capacitor_SMD:CP_Elec_3x5.3 -> Capacitor_SMD:C_0805_2012Metric_Pad1.18x1.45mm_HandSolder
- C5: renamed from C6; footprint Capacitor_SMD:CP_Elec_3x5.3 -> Capacitor_SMD:C_0805_2012Metric_Pad1.18x1.45mm_HandSolder
- C6: renamed from C7; value 100n -> 0.1u; footprint Capacitor_SMD:CP_Elec_3x5.3 -> Capacitor_SMD:C_0805_2012Metric_Pad1.18x1.45mm_HandSolder
- D1: footprint LED_THT:LED_D3.0mm_FlatTop -> LED_THT:LED_D5.0mm
- D3: renamed from D2; value 1N4001 -> 1N4002; footprint Diode_SMD:D_3220_8050Metric -> Diode_THT:D_DO-41_SOD81_P3.81mm_Vertical_AnodeUp
- D4: renamed from D3; value 1N4001 -> 1N4002; footprint Diode_SMD:D_3220_8050Metric -> Diode_THT:D_DO-41_SOD81_P3.81mm_Vertical_AnodeUp
- J1: footprint Connector_USB:USB_C_Receptacle_GCT_USB4135-GF-A_6P_TopMnt_Horizontal -> Connector_USB:USB_C_Receptacle_GCT_USB4125-xx-x-0190_6P_TopMnt_Horizontal
- J2, J3: footprint Connector_PinHeader_1.00mm:PinHeader_1x02_P1.00mm_Vertical -> Connector_PinHeader_2.54mm:PinHeader_1x02_P2.54mm_Vertical
- Q1: value 2N2219 -> 2N2222A; footprint Package_TO_SOT_THT:TO-39-3 -> Package_TO_SOT_THT:TO-92
- R1, R2: footprint Resistor_SMD:R_0603_1608Metric -> Resistor_SMD:R_0603_1608Metric_Pad0.98x0.95mm_HandSolder
- R10: renamed from R8; footprint Resistor_SMD:R_0603_1608Metric -> Resistor_SMD:R_0603_1608Metric_Pad0.98x0.95mm_HandSolder
- R11: renamed from R9; footprint Resistor_SMD:R_0603_1608Metric -> Resistor_SMD:R_0603_1608Metric_Pad0.98x0.95mm_HandSolder
- R12: renamed from R10; footprint Resistor_SMD:R_0603_1608Metric -> Resistor_SMD:R_0603_1608Metric_Pad0.98x0.95mm_HandSolder
- R13: value 1.2k -> 1k; footprint Resistor_SMD:R_0603_1608Metric -> Resistor_SMD:R_0603_1608Metric_Pad0.98x0.95mm_HandSolder
- R3: value 2.5k -> 2.52k; footprint Resistor_SMD:R_0603_1608Metric -> Resistor_SMD:R_0603_1608Metric_Pad0.98x0.95mm_HandSolder
- R4: value 820 -> 390; footprint Resistor_SMD:R_0603_1608Metric -> Resistor_SMD:R_0603_1608Metric_Pad0.98x0.95mm_HandSolder
- R5: value 510 -> 240; footprint Resistor_SMD:R_0603_1608Metric -> Resistor_SMD:R_0603_1608Metric_Pad0.98x0.95mm_HandSolder
- R6: renamed from R12; footprint Resistor_SMD:R_0603_1608Metric -> Resistor_SMD:R_0603_1608Metric_Pad0.98x0.95mm_HandSolder
- R7: renamed from R11; footprint Resistor_SMD:R_0603_1608Metric -> Resistor_SMD:R_0603_1608Metric_Pad0.98x0.95mm_HandSolder
- R8: renamed from R6; footprint Resistor_SMD:R_0603_1608Metric -> Resistor_SMD:R_0603_1608Metric_Pad0.98x0.95mm_HandSolder
- R9: renamed from R7; footprint Resistor_SMD:R_0603_1608Metric -> Resistor_SMD:R_0603_1608Metric_Pad0.98x0.95mm_HandSolder
- U1: value LM317_TO-220 -> LM317
- U3: renamed from U4; value NJM4560 -> NJM2904D; footprint NJM4560D:DIP762W46P254L880H425Q8 -> Package_DIP:DIP-8_W7.62mm_Socket
- renumbered U3 to U2, U5 to U4
Connections:
- net VDD is gone; now on net +5V: U3.8 (V+)
- net +5V: now also C1.1, D2.1 (K); no longer C2.1
- net GND: now also C1.2, J4.6 (Pin_6)
- net Pump: now also U2.14 (GPIO10); no longer U2.31 (GPIO26_ADC0)
- net SCL: now also J4.3 (Pin_3)
- net SDA: now also J4.2 (Pin_2)
- net +3V3 renamed +3.3V
- net +3.3V: now also C2.1, D2.2 (A), J4.1 (Pin_1)
- no-connect marks 35 -> 37
Other:
- moved on the sheet: C3, C4, C5, C6, D1, D3, D4, J1, J2, J3, Q1, Q2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
