File: bppy/PCB/BPN_2/BPN.kicad_pcb (KiCad board)
At the start: 2 copper layers, 57.6 x 54.1 mm, 35 parts, among them J1 USB_C_Receptacle_PowerOnly_6P, J2 Valve, J3 Pumpe, J4 Sensor_2, Q1 2N2222A, Q2 IRLIZ44N, U1 LM317, U2 Pico, U3 NJM2904D, U4 AMS6915

Commit message: PCB
Changed lines of the file:
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@@
     (property "ki_keywords" "R resistor")
     (attr smd)
-    (fp_text reference "R9" (at -0.05 -1.25) (layer "F.SilkS")
+    (fp_text reference "R9" (at 0.4275 -1.175) (layer "F.SilkS")
         (effects (font (size 1 1) (thickness 0.15)))
     )
