File: bppy/PCB/BPN_2/BPN.kicad_sch (KiCad schematic)
At the start: 35 parts, among them J1 USB_C_Receptacle_PowerOnly_6P, J2 Valve, J3 Pumpe, J4 Sensor_2, Q1 2N2222A, Q2 IRLIZ44N, U1 LM317, U2 Pico, U3 NJM2904D, U4 AMS6915

Commit message: PCB
Connections:
- net GND: now also C3.2, C4.2, R9.1
Changed lines of the file:
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@@
   (junction (at 210.82 51.435) (diameter 0) (color 0 0 0 0)
+  )
+  (junction (at 171.45 119.38) (diameter 0) (color 0 0 0 0)
   )
   (junction (at 150.495 61.595) (diameter 0) (color 0 0 0 0)
@@
         )
       )
+    )
+  )
+  (symbol (lib_name "GND_5") (lib_id "power:GND") (at 171.45 119.38 0) (unit 1)
+    (in_bom yes) (on_board yes) (dnp no) (fields_autoplaced)
+    (property "Reference" "#PWR025" (at 171.45 125.73 0)
+      (effects (font (size 1.27 1.27)) hide)
+    )
+    (property "Value" "GND" (at 171.45 124.46 0)
+      (effects (font (size 1.27 1.27)))
+    )
+    (property "Footprint" "" (at 171.45 119.38 0)
+      (effects (font (size 1.27 1.27)) hide)
+    )
+    (property "Datasheet" "" (at 171.45 119.38 0)
+      (effects (font (size 1.27 1.27)) hide)
+    )
+    (pin "1")
+    (instances
+      (project "BPN"
+        (path "/68ad6738-cf21-43e5-886f-0c54168215ea"
+          (reference "#PWR025") (unit 1)
+        )
+      )
