File: bppy/PCB/Differential/Differential.kicad_sch (KiCad schematic)
At the start: 26 parts, among them J1 USB_C_Receptacle_PowerOnly_6P, J3 Middle_Valve, J3 Pumpe, J4 Sensor_AMS, J4 Sensor_HX, Q2 IRLIZ44N, U1 LM317, U2 Pico

Commit message: PCB
Parts:
- added J8: UART, Connector_PinSocket_2.54mm:PinSocket_1x03_P2.54mm_Vertical, symbol Connector:Conn_01x03_Socket
- J3: value Pumpe -> Pump
- J4: footprint (none) -> Connector_PinSocket_2.54mm:PinSocket_1x04_P2.54mm_Vertical
Connections:
- net +3.3V: now also J4.1 (Pin_1), J4.2 (Pin_2)
- net GND: now also J8.3 (Pin_3)
- net TX: now reaches U2.1 (GPIO0)
- net TX: now also J8.1 (Pin_1)
- net RX: now reaches U2.2 (GPIO1)
- net RX: now also J8.2 (Pin_2)
- net Measurement_Valve renamed Cuff_Valve
- removed net Sensor_Power: J4.1 (Pin_1), J4.2 (Pin_2), U2.36 (3V3)
- no-connect marks 28 -> 27
