File: bppy/PCB/Differential/valve_control.kicad_sch (KiCad schematic)
At the start: 25 parts, among them J2 Valve, Q1 2N2222A, U2 NJM2114

Commit message: PCB
Parts:
- J2: value Valve -> Valve_Cuff
- J2: value Valve -> Valve_Baseline
- U3: renamed from U2; footprint (none) -> Package_DIP:DIP-8_W7.62mm
Connections:
- net Measurement_Valve renamed Cuff_Valve
Other:
- note added: "Cuff Valve Control Module"
- note removed: "Measurement Valve Control Module"
